File: minnowboard-to-busblaster.brd (EAGLE design)
At the start: 22 parts

Commit message: all
Parts:
- removed U$9: TLV3502-SOT23-8, minnowboard:SOT-23-8
- added D2: 1SMA5915BT3G, minnowboard:DIODE_SMB
- added R1: 20, resistor:R0805
- added U$4, U$6: SN74LV1T125, minnowboard:SC70-5
- R10, R17: value 10 -> 20000
- R12, R16: value 10 -> 30000
- R14, R5, R6, R7: value 10 -> 0
- moved D1 292.3 mm to (20.3, 35.6), turned to 90 degrees
- moved D5 288.6 mm to (24.1, 35.6), turned to 90 degrees
- moved R13 257.9 mm to (3.81, 26.7), turned to 90 degrees
- moved U$10 244.6 mm to (30.5, 21.6), turned to 270 degrees
- moved R17 215.5 mm to (29.2, 35.6), turned to 90 degrees
- moved R16 209.7 mm to (34.3, 35.6), turned to 270 degrees
- moved R14 189.6 mm to (68.6, 25.4), turned to 270 degrees
- moved R15 181.1 mm to (68.6, 10.2), turned to 270 degrees
- moved R12 173.9 mm to (39.4, 35.6), turned to 270 degrees
- moved R11 170.3 mm to (52.1, 35.6), turned to 90 degrees
- moved R10 162.4 mm to (44.5, 35.6), turned to 90 degrees
- moved R9 157.1 mm to (48.3, 35.6), turned to 270 degrees
- moved R7 146.7 mm to (68.6, 30.5), turned to 90 degrees
- moved R5 139.8 mm to (68.6, 35.6), turned to 270 degrees
- moved R8 138.6 mm to (68.6, 15.2), turned to 90 degrees
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Connections:
- new net N$1: JP1.1, JP1.2, R1.1
- net +3V3: now also D2.C, R1.2, U$4.5, U$6.5; no longer JP1.1, JP1.2, U$9.8
- net BB_DBGACK_R: now also U$6.4
- net BB_TDO_R: now also U$4.4
- net DBGACK_REF: now also U$6.2
- net GND: now also D2.A, U$4.1, U$4.3, U$6.1, U$6.3; no longer U$9.5
- net TDO_REF: now also U$4.2; no longer U$9.1
Routing:
- net GND: track 0.00 -> 33.7 mm
- net +3V3: track 0.00 -> 27.1 mm
- net BB_DBGACK: track 0.00 -> 10.8 mm
- net TDO_REF: track 0.00 -> 7.94 mm
- net +1V8: track 0.00 -> 7.50 mm
- net CMP_REF: track 0.00 -> 3.81 mm
- net BB_TDI_R: track 0.00 -> 2.75 mm
- net BB_TCLK_R: track 0.00 -> 2.75 mm
- net BB_DBGREQ_R: track 0.00 -> 2.43 mm
- net N$5: track 0.00 -> 2.42 mm
- net N$4: track 0.00 -> 2.32 mm
- net N$6: track 0.00 -> 2.11 mm
- net BB_TDO_R: track 0.00 -> 1.85 mm
- net N$3: track 0.00 -> 0.95 mm

Commit message: all
Parts:
- removed D1, D5: (no value), XUP_V1_04:DIODE_SOD323-W
- removed R10, R17: 20000, resistor:R0805
- removed R11, R9: 10, resistor:R0805
Connections:
- removed net CMP_REF: R11.2, R9.1
- removed net DBGACK_REF: D1.A, R10.1, R12.2, U$6.2
- removed net N$7: U$1.1, U$1.13, U$1.14, U$1.2, U$1.25, U$1.26, U$1.37, U$1.38, U$1.49, U$1.50, U$1.59, U$1.60
- removed net TDO_REF: D5.A, R16.2, R17.1, U$4.2
- net +3V3: no longer R11.1
- net DBGACK: now also R12.2, U$6.2; no longer D1.C
- net GND: now also U$1.1, U$1.13, U$1.14, U$1.2, U$1.25, U$1.26, U$1.37, U$1.38, U$1.49, U$1.50, U$1.59, U$1.60; no longer R10.2, R17.2, R9.2
- net TDO: now also R16.2, U$4.2; no longer D5.C
Routing:
- net TDO_REF: track 7.94 -> 0.00 mm
- net GND: track 33.7 -> 29.4 mm
- net CMP_REF: track 3.81 -> 0.00 mm
- net TDO: track 0.00 -> 2.86 mm
Other:
- board outline added: 72.4 x 35.6 mm

Commit message: all
Parts:
- removed R3: 10, resistor:R0805
- added TCLK1.8: 10, resistor:R0805
- DBGREF: value 10 -> 0
- TDO: value 0 -> 10
- turned DBGREF to 270 degrees
- turned TDI to 90 degrees
- renumbered JP1 to J2, R13 to TDI1.8, R14 to TDI, R15 to DBGACK, R2 to TMS1.8, R4 to DBGREF1.8, R5 to TCLK, R6 to TDO, R7 to TMS, R8 to DBGREF, U$1 to J1, U$10 to U1, U$4 to U3, U$6 to U2
Connections:
- net BB_DBGREQ: now also DBGREF.2; no longer TDI.2
- net BB_DBGREQ_R: now also DBGREF.1; no longer TDI.1
- net BB_TDI: now also TDI.2; no longer TMS.2
- net BB_TDI_R: now also TDI.1; no longer TMS.1
- net BB_TDO: now also TDO.2; no longer DBGREF.2
- net BB_TDO_R: now also TDO.1; no longer DBGREF.1
- net BB_TMS: now also TMS.2; no longer TDO.2
- net BB_TMS_R: now also TMS.1; no longer TDO.1
- net N$5: now also TCLK1.8.1; no longer R3.1
- net TCLK: now also TCLK1.8.2; no longer R3.2
Routing:
- net BB_DBGACK_R: track 0.00 -> 25.5 mm
- net BB_TDO_R: track 1.85 -> 26.7 mm
- net BB_TMS: track 0.00 -> 14.4 mm
- net BB_DBGACK: track 10.8 -> 0.00 mm
- net BB_TDI: track 0.00 -> 10.2 mm
- net BB_TDO: track 0.00 -> 9.80 mm
- net BB_DBGREQ: track 0.00 -> 9.75 mm
- net +1V8: track 7.50 -> 1.06 mm
- net TDO: track 2.86 -> 0.00 mm
- net N$1: track 0.00 -> 2.54 mm
- net BB_TMS_R: track 0.00 -> 2.43 mm
- net BB_DBGREQ_R: track 2.43 -> 0.00 mm
- net N$4: track 2.32 -> 0.00 mm
- net N$6: track 2.11 -> 0.00 mm
- net TCLK: track 0.00 -> 1.79 mm
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