File: minnowboard-to-busblaster.brd (EAGLE design)
At the start: 72.4 x 35.6 mm, 19 parts, among them J1 CIRCUITCO_MINNOW2_HIGH_SPEED, U1 SN74LV4T125, U2 SN74LV1T125, U3 SN74LV1T125

Commit message: all
Parts:
- added 1.8V, 5VSB, A0, A1, A2, A3, PLTRST, PMCRST, RSMRST, SCL, SDA: PAD-TESTPOINT, minnowboard:1,6/0,8
- moved TCLK1.8 14.6 mm to (3.81, 19.7)
- moved TDI1.8 9.52 mm to (3.81, 36.2)
- moved TMS1.8 9.52 mm to (3.81, 28.6)
- moved DBGREF 5.71 mm to (68.6, 9.53), turned to 90 degrees
- moved DBGACK 5.08 mm to (68.6, 15.2)
- moved R12 5.08 mm to (34.3, 35.6)
- moved R16 5.08 mm to (39.4, 35.6), turned to 90 degrees
Connections:
- new net N$11: A1.1, J1.33
- new net N$13: J1.41, RSMRST.1
- new net N$14: A3.1, J1.36
- new net N$15: J1.21, SCL.1
- new net N$16: J1.23, SDA.1
- new net N$7: 5VSB.1, J1.7
- new net N$8: A2.1, J1.35
- new net N$9: A0.1, J1.34
- net +1V8: now also 1.8V.1
- net GND: now also J2.18, J2.20
- net N$23: now also J1.46, PMCRST.1; no longer J2.18
- net N$24: now also J1.47, PLTRST.1; no longer J2.20
Routing:
- net GND: track 28.7 -> 174.6 mm, vias 0 -> 9
- net BB_TCLK_R: track 1.89 -> 58.1 mm, vias 0 -> 2
- net BB_TMS_R: track 2.43 -> 50.4 mm
- net DBGACK: track 0.00 -> 46.8 mm, vias 0 -> 2
- net +1V8: track 1.06 -> 46.9 mm, vias 0 -> 2
- net BB_DBGREQ_R: track 0.00 -> 43.8 mm
- net N$5: track 1.06 -> 43.4 mm
- net TDO: track 0.00 -> 38.9 mm
- net BB_TDI_R: track 2.22 -> 39.0 mm
- net N$4: track 0.00 -> 36.7 mm, vias 0 -> 2
- net N$6: track 0.00 -> 33.2 mm, vias 0 -> 2
- net N$3: track 0.00 -> 29.4 mm, vias 0 -> 2
- net N$1: track 2.54 -> 30.7 mm, vias 0 -> 1
- net DBGREQ: track 0.00 -> 20.2 mm
- net BB_TCLK: track 0.00 -> 17.2 mm, vias 0 -> 1
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Other:
- board size 72.4 x 35.6 mm -> 71.8 x 34.3 mm

Commit message: all
Parts:
- removed 1.8V, 5VSB, A0, A1, A2, A3, PLTRST, PMCRST, RSMRST, SCL, SDA: PAD-TESTPOINT, minnowboard:1,6/0,8
- moved TMS 50.2 mm to (18.4, 29.2), turned to 180 degrees
- moved TDI 45.5 mm to (24.1, 34.9)
- moved DBGREF 43.3 mm to (31.8, 32.4), turned to 0 degrees
- moved DBGACK 38.6 mm to (30.5, 8.89), turned to 0 degrees
- moved TDO 38.5 mm to (30.5, 14.6), turned to 0 degrees
- moved TCLK 37.7 mm to (31.8, 27.3), turned to 0 degrees
- moved DBGREF1.8 34.2 mm to (31.8, 29.8), turned to 0 degrees
- moved R12 30.1 mm to (20.3, 8.89), turned to 180 degrees
- moved R16 28.3 mm to (20.3, 14.6), turned to 0 degrees
- moved U3 24.3 mm to (25.4, 14.6)
- moved U2 23.3 mm to (25.4, 8.89)
- moved TCLK1.8 22.7 mm to (26.0, 24.1), turned to 270 degrees
- moved R1 20.7 mm to (33.7, 18.4)
- moved D2 18.5 mm to (27.3, 18.4)
- moved J2 15.9 mm to (45.1, 22.9)
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Connections:
- net +1V8: no longer 1.8V.1
- net N$11: no longer A1.1
- net N$13: no longer RSMRST.1
- net N$14: no longer A3.1
- net N$15: no longer SCL.1
- net N$16: no longer SDA.1
- net N$23: no longer PMCRST.1
- net N$24: no longer PLTRST.1
- net N$7: no longer 5VSB.1
- net N$8: no longer A2.1
- net N$9: no longer A0.1
Routing:
- net BB_TCLK_R: track 58.1 -> 4.11 mm, vias 2 -> 0
- net BB_TMS_R: track 50.4 -> 5.18 mm
- net N$5: track 43.4 -> 2.48 mm
- net BB_DBGREQ_R: track 43.8 -> 4.74 mm
- net BB_TDI_R: track 39.0 -> 6.87 mm
- net N$4: track 36.7 -> 4.98 mm, vias 2 -> 0
- net N$6: track 33.2 -> 3.96 mm, vias 2 -> 0
- net BB_TDO_R: track 32.3 -> 3.30 mm, vias 2 -> 0
- net N$3: track 29.4 -> 5.01 mm, vias 2 -> 0
- net BB_TMS: track 12.3 -> 35.0 mm, vias 0 -> 2
- net DBGREQ: track 20.2 -> 41.4 mm, vias 0 -> 2
- net BB_DBGACK_R: track 24.2 -> 3.33 mm
- net TDI: track 7.62 -> 26.6 mm, vias 0 -> 2
- net BB_DBGREQ: track 14.2 -> 29.5 mm, vias 0 -> 2
- net TMS: track 8.51 -> 21.4 mm, vias 0 -> 2
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Other:
- board size 71.8 x 34.3 mm -> 48.9 x 34.9 mm

Commit message: all
Parts:
- added A0, A1, A2, A3, U$1: TESTPAD, minnowboard:TESTPAD
Connections:
- removed net N$13: J1.41
- new net RMRST: J1.41, U$1.P$1
- net N$11: now also A1.P$1
- net N$14: now also A3.P$1
- net N$8: now also A2.P$1
- net N$9: now also A0.P$1
Routing:
- net GND: track 165.3 -> 190.6 mm, vias 8 -> 7
- net +1V8: track 59.6 -> 67.6 mm
- net TDO: track 29.4 -> 36.2 mm
- net RMRST: track 0.00 -> 4.99 mm
- net N$8: track 0.00 -> 3.54 mm
- net N$14: track 0.00 -> 3.18 mm
- net N$11: track 0.00 -> 2.98 mm
- net N$9: track 0.00 -> 2.94 mm
- net DBGACK: track 34.8 -> 37.5 mm, vias 0 -> 2
- net N$1: track 27.8 -> 26.5 mm, vias 0 -> 1
- net DBGREQ: track 41.4 -> 42.6 mm
- net TCLK: track 26.3 -> 25.7 mm

Commit message: all
Parts:
- removed DBGREF1.8: 10, resistor:R0805
Connections:
- net DBGREQ: no longer DBGREF1.8.2
- net N$6: no longer DBGREF1.8.1
Routing:
- net DBGREQ: track 42.6 -> 38.4 mm
- net N$6: track 3.96 -> 2.37 mm
Changed lines of the file:
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@@
 <element name="TMS1.8" library="resistor" package="R0805" value="10" x="18.415" y="26.67" rot="R180"/>
 <element name="TCLK1.8" library="resistor" package="R0805" value="10" x="26.035" y="24.13" rot="R270"/>
-<element name="DBGREF1.8" library="resistor" package="R0805" value="10" x="31.75" y="29.845"/>
 <element name="TCLK" library="resistor" package="R0805" value="0" x="31.75" y="27.305"/>
 <element name="TMS" library="resistor" package="R0805" value="0" x="18.415" y="29.21" rot="R180"/>
@@
 <signal name="DBGREQ">
 <contactref element="J1" pad="40"/>
-<contactref element="DBGREF1.8" pad="2"/>
-<wire x1="32.7" y1="29.845" x2="36.83" y2="29.845" width="0.3" layer="1"/>
 <via x="36.83" y="29.845" extent="1-16" drill="0.6"/>
 <wire x1="36.83" y1="29.845" x2="36.83" y2="26.67" width="0.3" layer="16"/>
@@
 </signal>
 <signal name="N$6">
-<contactref element="DBGREF1.8" pad="1"/>
 <contactref element="U1" pad="11"/>
 <wire x1="27.1" y1="29.21" x2="28.575" y2="29.21" width="0.3" layer="1"/>
 <wire x1="28.575" y1="29.21" x2="29.21" y2="29.845" width="0.3" layer="1"/>
-<wire x1="29.21" y1="29.845" x2="30.8" y2="29.845" width="0.3" layer="1"/>
 </signal>
 <signal name="N$1">
