File: minnowboard-to-busblaster.sch (EAGLE design)
At the start: 22 parts

Commit message: all
Parts:
- removed U$9: TLV3502-SOT23-8, minnowboard:TLV3502-SOT23-8
- added D2: 1SMA5915BT3G, minnowboard:DIODE_ZENER-DIODESMB
- added R1: 20, resistor:R-EU_R0805
- added U$4, U$6: SN74LV1T125, minnowboard:SN74LV1T125
- R10, R17: value 10 -> 20000
- R12, R16: value 10 -> 30000
- R14, R5, R6, R7: value 10 -> 0
Connections:
- new net N$1: JP1.1, JP1.2, R1.1
- net +3V3: now also D2.C, R1.2, U$4.VCC, U$6.VCC; no longer JP1.1, JP1.2, U$9.V+
- net BB_DBGACK_R: now also U$6.Y
- net BB_TDO_R: now also U$4.Y
- net DBGACK_REF: now also U$6.A
- net GND: now also D2.A, U$4.GND, U$4.OE, U$6.GND, U$6.OE; no longer U$9.V-
- net TDO_REF: now also U$4.A; no longer U$9.+INA
Other:
- moved on the sheet: D5, R11, R13, R16, R17, R2, R3, R4, R9

Commit message: all
Parts:
- removed D1, D5: (no value), XUP_V1_04:DIODE_DIODE-SOD323-W
- removed R10, R17: 20000, resistor:R-EU_R0805
- removed R11, R9: 10, resistor:R-EU_R0805
Connections:
- removed net CMP_REF: R11.2, R9.1
- removed net DBGACK_REF: D1.A, R10.1, R12.2, U$6.A
- removed net N$7: U$1.GND@1, U$1.GND@10, U$1.GND@11, U$1.GND@12, U$1.GND@2, U$1.GND@3, U$1.GND@4, U$1.GND@5, U$1.GND@6, U$1.GND@7, U$1.GND@8, U$1.GND@9
- removed net TDO_REF: D5.A, R16.2, R17.1, U$4.A
- net +3V3: no longer R11.1
- net DBGACK: now also R12.2, U$6.A; no longer D1.C
- net GND: now also U$1.GND@1, U$1.GND@10, U$1.GND@11, U$1.GND@12, U$1.GND@2, U$1.GND@3, U$1.GND@4, U$1.GND@5, U$1.GND@6, U$1.GND@7, U$1.GND@8, U$1.GND@9; no longer R10.2, R17.2, R9.2
- net TDO: now also R16.2, U$4.A; no longer D5.C
Other:
- moved on the sheet: R12, R16

Commit message: all
Parts:
- renumbered JP1 to J2, R13 to TDI1.8, R14 to DBGREF, R15 to DBGACK, R2 to TMS1.8, R3 to TCLK1.8, R4 to DBGREF1.8, R5 to TCLK, R6 to TMS, R7 to TDI, R8 to TDO, U$1 to J1, U$10 to U1, U$4 to U3, U$6 to U2

Commit message: all
Parts:
- added 1.8V, 5VSB, A0, A1, A2, A3, PLTRST, PMCRST, RSMRST, SCL, SDA: PAD-TESTPOINT, minnowboard:PAD-TESTPOINT
Connections:
- new net N$11: A1.P, J1.XDP_H_OBSDATA_A1
- new net N$13: J1.HOOK0, RSMRST.P
- new net N$14: A3.P, J1.XDP_H_OBSDATA_A3
- new net N$15: J1.EXP_I2C_SCL, SCL.P
- new net N$16: J1.EXP_I2C_SDA, SDA.P
- new net N$7: 5VSB.P, J1.5VSB@1
- new net N$8: A2.P, J1.XDP_H_OBSDATA_A2
- new net N$9: A0.P, J1.XDP_H_OBSDATA_A0
- net +1V8: now also 1.8V.P
- net GND: now also J2.18, J2.20
- net N$23: now also J1.HOOK7, PMCRST.P; no longer J2.18
- net N$24: now also J1.HOOK6, PLTRST.P; no longer J2.20
Changed lines of the file:
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@@
 <setting verticaltext="up"/>
 </settings>
-<grid distance="0.1" unitdist="inch" unit="inch" style="lines" multiple="1" display="yes" altdistance="0.01" altunitdist="inch" altunit="inch"/>
+<grid distance="0.1" unitdist="inch" unit="mm" style="lines" multiple="1" display="yes" altdistance="0.01" altunitdist="inch" altunit="inch"/>
 <layers>
 <layer number="1" name="Top" color="4" fill="1" visible="no" active="no"/>
@@
 <part name="GND7" library="supply1" deviceset="GND" device=""/>
 <part name="GND1" library="supply1" deviceset="GND" device=""/>
+<part name="A0" library="minnowboard" deviceset="PAD-TESTPOINT" device=""/>
+<part name="A1" library="minnowboard" deviceset="PAD-TESTPOINT" device=""/>
+<part name="A2" library="minnowboard" deviceset="PAD-TESTPOINT" device=""/>
+<part name="A3" library="minnowboard" deviceset="PAD-TESTPOINT" device=""/>
+<part name="5VSB" library="minnowboard" deviceset="PAD-TESTPOINT" device=""/>
+<part name="1.8V" library="minnowboard" deviceset="PAD-TESTPOINT" device=""/>
+<part name="SCL" library="minnowboard" deviceset="PAD-TESTPOINT" device=""/>
+<part name="SDA" library="minnowboard" deviceset="PAD-TESTPOINT" device=""/>
+<part name="RSMRST" library="minnowboard" deviceset="PAD-TESTPOINT" device=""/>
+<part name="PLTRST" library="minnowboard" deviceset="PAD-TESTPOINT" device=""/>
+<part name="PMCRST" library="minnowboard" deviceset="PAD-TESTPOINT" device=""/>
 </parts>
 <sheets>
@@
 <instance part="J1" gate="G$1" x="-5.08" y="50.8"/>
 <instance part="J2" gate="A" x="182.88" y="55.88"/>
-<instance part="U$2" gate="G$1" x="25.4" y="88.9" rot="R270"/>
+<instance part="U$2" gate="G$1" x="22.86" y="88.9" rot="R270"/>
 <instance part="U$5" gate="G$1" x="101.6" y="7.62" rot="MR90"/>
 <instance part="TMS1.8" gate="G$1" x="66.04" y="33.02" rot="MR0"/>
@@
 <instance part="GND7" gate="1" x="86.36" y="78.74" rot="MR0"/>
 <instance part="GND1" gate="1" x="-38.1" y="5.08" rot="MR0"/>
+<instance part="A0" gate="P" x="30.48" y="22.86" rot="R180"/>
+<instance part="A1" gate="P" x="30.48" y="20.32" rot="R180"/>
+<instance part="A2" gate="P" x="30.48" y="17.78" rot="R180"/>
+<instance part="A3" gate="P" x="30.48" y="15.24" rot="R180"/>
+<instance part="5VSB" gate="P" x="-40.64" y="88.9"/>
+<instance part="1.8V" gate="P" x="30.48" y="88.9" rot="R180"/>
+<instance part="SCL" gate="P" x="30.48" y="66.04" rot="R180"/>
+<instance part="SDA" gate="P" x="30.48" y="63.5" rot="R180"/>
+<instance part="RSMRST" gate="P" x="30.48" y="60.96" rot="R180"/>
+<instance part="PLTRST" gate="P" x="30.48" y="45.72" rot="R180"/>
+<instance part="PMCRST" gate="P" x="30.48" y="43.18" rot="R180"/>
 </instances>
 <busses>
@@
 <wire x1="-33.02" y1="15.24" x2="-38.1" y2="15.24" width="0.1524" layer="91"/>
 <pinref part="GND1" gate="1" pin="GND"/>
+<wire x1="-38.1" y1="43.18" x2="-40.64" y2="43.18" width="0.1524" layer="91"/>
+</segment>
+<segment>
+<pinref part="J2" gate="A" pin="20"/>
+<wire x1="187.96" y1="43.18" x2="198.12" y2="43.18" width="0.1524" layer="91"/>
+</segment>
+<segment>
+<pinref part="J2" gate="A" pin="18"/>
+<wire x1="187.96" y1="45.72" x2="198.12" y2="45.72" width="0.1524" layer="91"/>
 </segment>
 </net>
@@
 <segment>
 <pinref part="J1" gate="G$1" pin="V1P8A@1"/>
-<wire x1="20.32" y1="88.9" x2="22.86" y2="88.9" width="0.1524" layer="91"/>
 <pinref part="U$2" gate="G$1" pin="+1V8"/>
-<junction x="22.86" y="88.9"/>
+<wire x1="27.94" y1="88.9" x2="20.32" y2="88.9" width="0.1524" layer="91"/>
+<pinref part="1.8V" gate="P" pin="P"/>
 </segment>
 <segment>
@@
 <pinref part="J2" gate="A" pin="16"/>
 <wire x1="187.96" y1="48.26" x2="198.12" y2="48.26" width="0.1524" layer="91"/>
-</segment>
-</net>
-<net name="N$23" class="0">
-<segment>
-<pinref part="J2" gate="A" pin="18"/>
-<wire x1="187.96" y1="45.72" x2="198.12" y2="45.72" width="0.1524" layer="91"/>
-</segment>
-</net>
-<net name="N$24" class="0">
-<segment>
-<pinref part="J2" gate="A" pin="20"/>
-<wire x1="187.96" y1="43.18" x2="198.12" y2="43.18" width="0.1524" layer="91"/>
 </segment>
 </net>
@@
 </segment>
 </net>
+<net name="N$7" class="0">
+<segment>
+<pinref part="J1" gate="G$1" pin="5VSB@1"/>
+<wire x1="-33.02" y1="88.9" x2="-38.1" y2="88.9" width="0.1524" layer="91"/>
+<pinref part="5VSB" gate="P" pin="P"/>
+</segment>
+</net>
+<net name="N$9" class="0">
+<segment>
+<pinref part="J1" gate="G$1" pin="XDP_H_OBSDATA_A0"/>
+<wire x1="27.94" y1="22.86" x2="20.32" y2="22.86" width="0.1524" layer="91"/>
+<pinref part="A0" gate="P" pin="P"/>
+</segment>
+</net>
+<net name="N$11" class="0">
+<segment>
+<pinref part="J1" gate="G$1" pin="XDP_H_OBSDATA_A1"/>
+<wire x1="27.94" y1="20.32" x2="20.32" y2="20.32" width="0.1524" layer="91"/>
+<pinref part="A1" gate="P" pin="P"/>
+</segment>
+</net>
+<net name="N$14" class="0">
+<segment>
+<pinref part="J1" gate="G$1" pin="XDP_H_OBSDATA_A3"/>
+<wire x1="27.94" y1="15.24" x2="20.32" y2="15.24" width="0.1524" layer="91"/>
+<pinref part="A3" gate="P" pin="P"/>
+</segment>
+</net>
+<net name="N$15" class="0">
+<segment>
+<pinref part="J1" gate="G$1" pin="EXP_I2C_SCL"/>
+<wire x1="20.32" y1="66.04" x2="27.94" y2="66.04" width="0.1524" layer="91"/>
+<pinref part="SCL" gate="P" pin="P"/>
+</segment>
+</net>
+<net name="N$16" class="0">
+<segment>
+<pinref part="J1" gate="G$1" pin="EXP_I2C_SDA"/>
+<wire x1="20.32" y1="63.5" x2="27.94" y2="63.5" width="0.1524" layer="91"/>
+<pinref part="SDA" gate="P" pin="P"/>
+</segment>
+</net>
+<net name="N$8" class="0">
+<segment>
+<pinref part="J1" gate="G$1" pin="XDP_H_OBSDATA_A2"/>
+<pinref part="A2" gate="P" pin="P"/>
+<wire x1="20.32" y1="17.78" x2="27.94" y2="17.78" width="0.4064" layer="91"/>
+</segment>
+</net>
+<net name="N$13" class="0">
+<segment>
+<pinref part="J1" gate="G$1" pin="HOOK0"/>
+<wire x1="20.32" y1="60.96" x2="27.94" y2="60.96" width="0.254" layer="91"/>
+<pinref part="RSMRST" gate="P" pin="P"/>
+</segment>
+</net>
+<net name="N$24" class="0">
+<segment>
+<pinref part="J1" gate="G$1" pin="HOOK6"/>
+<wire x1="20.32" y1="45.72" x2="27.94" y2="45.72" width="0.254" layer="91"/>
+<pinref part="PLTRST" gate="P" pin="P"/>
+</segment>
+</net>
+<net name="N$23" class="0">
+<segment>
+<pinref part="J1" gate="G$1" pin="HOOK7"/>
+<wire x1="20.32" y1="43.18" x2="27.94" y2="43.18" width="0.254" layer="91"/>
+<pinref part="PMCRST" gate="P" pin="P"/>
+</segment>
+</net>

Commit message: all
Parts:
- removed 1.8V, 5VSB, A0, A1, A2, A3, PLTRST, PMCRST, RSMRST, SCL, SDA: PAD-TESTPOINT, minnowboard:PAD-TESTPOINT
Connections:
- net +1V8: no longer 1.8V.P
- net N$11: no longer A1.P
- net N$13: no longer RSMRST.P
- net N$14: no longer A3.P
- net N$15: no longer SCL.P
- net N$16: no longer SDA.P
- net N$23: no longer PMCRST.P
- net N$24: no longer PLTRST.P
- net N$7: no longer 5VSB.P
- net N$8: no longer A2.P
- net N$9: no longer A0.P
Changed lines of the file:
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@@
 <setting verticaltext="up"/>
 </settings>
-<grid distance="0.1" unitdist="inch" unit="mm" style="lines" multiple="1" display="yes" altdistance="0.01" altunitdist="inch" altunit="inch"/>
+<grid distance="0.1" unitdist="inch" unit="inch" style="lines" multiple="1" display="yes" altdistance="0.01" altunitdist="inch" altunit="inch"/>
 <layers>
 <layer number="1" name="Top" color="4" fill="1" visible="no" active="no"/>
@@
 <part name="GND7" library="supply1" deviceset="GND" device=""/>
 <part name="GND1" library="supply1" deviceset="GND" device=""/>
-<part name="A0" library="minnowboard" deviceset="PAD-TESTPOINT" device=""/>
-<part name="A1" library="minnowboard" deviceset="PAD-TESTPOINT" device=""/>
-<part name="A2" library="minnowboard" deviceset="PAD-TESTPOINT" device=""/>
-<part name="A3" library="minnowboard" deviceset="PAD-TESTPOINT" device=""/>
-<part name="5VSB" library="minnowboard" deviceset="PAD-TESTPOINT" device=""/>
-<part name="1.8V" library="minnowboard" deviceset="PAD-TESTPOINT" device=""/>
-<part name="SCL" library="minnowboard" deviceset="PAD-TESTPOINT" device=""/>
-<part name="SDA" library="minnowboard" deviceset="PAD-TESTPOINT" device=""/>
-<part name="RSMRST" library="minnowboard" deviceset="PAD-TESTPOINT" device=""/>
-<part name="PLTRST" library="minnowboard" deviceset="PAD-TESTPOINT" device=""/>
-<part name="PMCRST" library="minnowboard" deviceset="PAD-TESTPOINT" device=""/>
 </parts>
 <sheets>
@@
 <instance part="GND7" gate="1" x="86.36" y="78.74" rot="MR0"/>
 <instance part="GND1" gate="1" x="-38.1" y="5.08" rot="MR0"/>
-<instance part="A0" gate="P" x="30.48" y="22.86" rot="R180"/>
-<instance part="A1" gate="P" x="30.48" y="20.32" rot="R180"/>
-<instance part="A2" gate="P" x="30.48" y="17.78" rot="R180"/>
-<instance part="A3" gate="P" x="30.48" y="15.24" rot="R180"/>
-<instance part="5VSB" gate="P" x="-40.64" y="88.9"/>
-<instance part="1.8V" gate="P" x="30.48" y="88.9" rot="R180"/>
-<instance part="SCL" gate="P" x="30.48" y="66.04" rot="R180"/>
-<instance part="SDA" gate="P" x="30.48" y="63.5" rot="R180"/>
-<instance part="RSMRST" gate="P" x="30.48" y="60.96" rot="R180"/>
-<instance part="PLTRST" gate="P" x="30.48" y="45.72" rot="R180"/>
-<instance part="PMCRST" gate="P" x="30.48" y="43.18" rot="R180"/>
 </instances>
 <busses>
@@
 <pinref part="U$2" gate="G$1" pin="+1V8"/>
 <wire x1="27.94" y1="88.9" x2="20.32" y2="88.9" width="0.1524" layer="91"/>
-<pinref part="1.8V" gate="P" pin="P"/>
 </segment>
 <segment>
@@
 <pinref part="J1" gate="G$1" pin="5VSB@1"/>
 <wire x1="-33.02" y1="88.9" x2="-38.1" y2="88.9" width="0.1524" layer="91"/>
-<pinref part="5VSB" gate="P" pin="P"/>
 </segment>
 </net>
@@
 <pinref part="J1" gate="G$1" pin="XDP_H_OBSDATA_A0"/>
 <wire x1="27.94" y1="22.86" x2="20.32" y2="22.86" width="0.1524" layer="91"/>
-<pinref part="A0" gate="P" pin="P"/>
 </segment>
 </net>
@@
 <pinref part="J1" gate="G$1" pin="XDP_H_OBSDATA_A1"/>
 <wire x1="27.94" y1="20.32" x2="20.32" y2="20.32" width="0.1524" layer="91"/>
-<pinref part="A1" gate="P" pin="P"/>
 </segment>
 </net>
@@
 <pinref part="J1" gate="G$1" pin="XDP_H_OBSDATA_A3"/>
 <wire x1="27.94" y1="15.24" x2="20.32" y2="15.24" width="0.1524" layer="91"/>
-<pinref part="A3" gate="P" pin="P"/>
 </segment>
 </net>
@@
 <pinref part="J1" gate="G$1" pin="EXP_I2C_SCL"/>
 <wire x1="20.32" y1="66.04" x2="27.94" y2="66.04" width="0.1524" layer="91"/>
-<pinref part="SCL" gate="P" pin="P"/>
 </segment>
 </net>
@@
 <pinref part="J1" gate="G$1" pin="EXP_I2C_SDA"/>
 <wire x1="20.32" y1="63.5" x2="27.94" y2="63.5" width="0.1524" layer="91"/>
-<pinref part="SDA" gate="P" pin="P"/>
 </segment>
 </net>
@@
 <segment>
 <pinref part="J1" gate="G$1" pin="XDP_H_OBSDATA_A2"/>
-<pinref part="A2" gate="P" pin="P"/>
 <wire x1="20.32" y1="17.78" x2="27.94" y2="17.78" width="0.4064" layer="91"/>
 </segment>
@@
 <pinref part="J1" gate="G$1" pin="HOOK0"/>
 <wire x1="20.32" y1="60.96" x2="27.94" y2="60.96" width="0.254" layer="91"/>
-<pinref part="RSMRST" gate="P" pin="P"/>
 </segment>
 </net>
@@
 <pinref part="J1" gate="G$1" pin="HOOK6"/>
 <wire x1="20.32" y1="45.72" x2="27.94" y2="45.72" width="0.254" layer="91"/>
-<pinref part="PLTRST" gate="P" pin="P"/>
 </segment>
 </net>
@@
 <pinref part="J1" gate="G$1" pin="HOOK7"/>
 <wire x1="20.32" y1="43.18" x2="27.94" y2="43.18" width="0.254" layer="91"/>
-<pinref part="PMCRST" gate="P" pin="P"/>
-</segment>
-</net>
+</segment>
+</net>

Commit message: all
Parts:
- added A0, A1, A2, A3, U$1: TESTPAD, minnowboard:TESTPAD
Connections:
- removed net N$13: J1.HOOK0
- new net RMRST: J1.HOOK0, U$1.TESTPAD
- net N$11: now also A1.TESTPAD
- net N$14: now also A3.TESTPAD
- net N$8: now also A2.TESTPAD
- net N$9: now also A0.TESTPAD
Changed lines of the file:
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@@
 <part name="GND7" library="supply1" deviceset="GND" device=""/>
 <part name="GND1" library="supply1" deviceset="GND" device=""/>
+<part name="U$1" library="minnowboard" deviceset="TESTPAD" device=""/>
+<part name="A0" library="minnowboard" deviceset="TESTPAD" device=""/>
+<part name="A1" library="minnowboard" deviceset="TESTPAD" device=""/>
+<part name="A2" library="minnowboard" deviceset="TESTPAD" device=""/>
+<part name="A3" library="minnowboard" deviceset="TESTPAD" device=""/>
 </parts>
 <sheets>
@@
 <instance part="GND7" gate="1" x="86.36" y="78.74" rot="MR0"/>
 <instance part="GND1" gate="1" x="-38.1" y="5.08" rot="MR0"/>
+<instance part="U$1" gate="G$1" x="25.4" y="60.96"/>
+<instance part="A0" gate="G$1" x="25.4" y="22.86"/>
+<instance part="A1" gate="G$1" x="25.4" y="20.32"/>
+<instance part="A2" gate="G$1" x="25.4" y="17.78"/>
+<instance part="A3" gate="G$1" x="25.4" y="15.24"/>
 </instances>
 <busses>
@@
 <segment>
 <pinref part="J1" gate="G$1" pin="XDP_H_OBSDATA_A0"/>
-<wire x1="27.94" y1="22.86" x2="20.32" y2="22.86" width="0.1524" layer="91"/>
+<pinref part="A0" gate="G$1" pin="TESTPAD"/>
+<wire x1="25.4" y1="22.86" x2="20.32" y2="22.86" width="0.1524" layer="91"/>
 </segment>
 </net>
@@
 <segment>
 <pinref part="J1" gate="G$1" pin="XDP_H_OBSDATA_A1"/>
-<wire x1="27.94" y1="20.32" x2="20.32" y2="20.32" width="0.1524" layer="91"/>
+<pinref part="A1" gate="G$1" pin="TESTPAD"/>
+<wire x1="25.4" y1="20.32" x2="20.32" y2="20.32" width="0.1524" layer="91"/>
 </segment>
 </net>
@@
 <segment>
 <pinref part="J1" gate="G$1" pin="XDP_H_OBSDATA_A3"/>
-<wire x1="27.94" y1="15.24" x2="20.32" y2="15.24" width="0.1524" layer="91"/>
+<pinref part="A3" gate="G$1" pin="TESTPAD"/>
+<wire x1="25.4" y1="15.24" x2="20.32" y2="15.24" width="0.1524" layer="91"/>
 </segment>
 </net>
@@
 <segment>
 <pinref part="J1" gate="G$1" pin="XDP_H_OBSDATA_A2"/>
-<wire x1="20.32" y1="17.78" x2="27.94" y2="17.78" width="0.4064" layer="91"/>
-</segment>
-</net>
-<net name="N$13" class="0">
+<wire x1="20.32" y1="17.78" x2="25.4" y2="17.78" width="0.4064" layer="91"/>
+<pinref part="A2" gate="G$1" pin="TESTPAD"/>
+</segment>
+</net>
+<net name="RMRST" class="0">
 <segment>
 <pinref part="J1" gate="G$1" pin="HOOK0"/>
-<wire x1="20.32" y1="60.96" x2="27.94" y2="60.96" width="0.254" layer="91"/>
-</segment>
-</net>
+<wire x1="20.32" y1="60.96" x2="25.4" y2="60.96" width="0.254" layer="91"/>
+<pinref part="U$1" gate="G$1" pin="TESTPAD"/>
+</segment>
+</net>

Commit message: all
Parts:
- removed DBGREF1.8: 10, resistor:R-EU_R0805
Connections:
- net DBGREQ: no longer DBGREF1.8.2
- net N$6: no longer DBGREF1.8.1
Changed lines of the file:
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@@
 <part name="TMS1.8" library="resistor" deviceset="R-EU_" device="R0805" value="10"/>
 <part name="TCLK1.8" library="resistor" deviceset="R-EU_" device="R0805" value="10"/>
-<part name="DBGREF1.8" library="resistor" deviceset="R-EU_" device="R0805" value="10"/>
 <part name="GND5" library="supply1" deviceset="GND" device=""/>
 <part name="TCLK" library="resistor" deviceset="R-EU_" device="R0805" value="0"/>
@@
 <instance part="TMS1.8" gate="G$1" x="66.04" y="33.02" rot="MR0"/>
 <instance part="TCLK1.8" gate="G$1" x="66.04" y="22.86" rot="R180"/>
-<instance part="DBGREF1.8" gate="G$1" x="66.04" y="12.7" rot="MR0"/>
 <instance part="GND5" gate="1" x="198.12" y="38.1"/>
 <instance part="TCLK" gate="G$1" x="162.56" y="55.88"/>
@@
 </segment>
 <segment>
-<pinref part="DBGREF1.8" gate="G$1" pin="2"/>
 <wire x1="60.96" y1="12.7" x2="53.34" y2="12.7" width="0.1524" layer="91"/>
 <label x="53.34" y="12.7" size="1.778" layer="95"/>
@@
 <net name="N$6" class="0">
 <segment>
-<pinref part="DBGREF1.8" gate="G$1" pin="1"/>
 <wire x1="71.12" y1="12.7" x2="76.2" y2="12.7" width="0.1524" layer="91"/>
 <pinref part="U1" gate="G$1" pin="4Y"/>
